File: PowerModule_PTH_XT30M.kicad_pcb (KiCad board)
At the start: 2 copper layers, 26.3 x 20 mm, 5 parts, among them J1 Conn_01x05, J2 Conn_01x05, J3 XT30PW-M

Commit message: Fix module name text
Other:
- board text added: "PnP Power Module XT30 Male"
- board text removed: "PnP Power Module XT30 Female"
Changed lines of the file:
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@@
 		(layer "Edge.Cuts")
 	)
-	(gr_text "PnP Power Module\nXT30 Female"
+	(gr_text "PnP Power Module\nXT30 Male"
 		(at 142.685 89.5 0)
 		(layer "B.SilkS")
