File: panel.kicad_pcb (KiCad board)
At the start: 2 copper layers, 92.8 x 74 mm, 57 parts, among them J1 Conn_01x05, J2 Conn_01x05, J3 XT30PW-M

Commit message: Fix module name text
Other:
- board text added: "PnP Power Module XT30 Male"
- board text removed: "PnP Power Module XT30 Female"
